File: pcb/iceGDROM/iceGDROM.sch (KiCad schematic (older format))
At the start: 82 parts, among them CN1 Molex_52602_0579, J1 Conn_02x22_Odd_Even, J2 Micro_SD_Card_Det_Hirose_DM3AT, U1 ICE40HX8K-BG121, U2 ME6206A25M3G_SOT23, U3 LD1117S12TR_SOT223, U4 W25Q32JVSS, X1 SG-310SCF

Commit message: Included the SPI Memory card into the schematic as a major point. Created a footprint for the tactile button being used and including the 3D model due to no NC clause.
Parts:
- removed R2, R4: R, Resistor_SMD:R_0603_1608Metric, symbol Device:R
- removed SW?: SW_Push, symbol Switch:SW_Push
- added C1: 100n, Capacitor_SMD:C_0603_1608Metric, symbol Device:C
- added R1, R10, R11, R12, R13, R9: 10K, Resistor_SMD:R_0603_1608Metric, symbol Device:R
- added SW1, SW2, SW3: SW_Push, iceGDROM:SW_Push_SPST_NO_Alps_SKRP, symbol Switch:SW_Push
- added TP17, TP18, TP21, TP22, TP23, TP24, TP25, TP26, TP27, TP28, TP29: TestPoint, TestPoint:TestPoint_Pad_D1.0mm, symbol Connector:TestPoint
- J3: renamed from J?; footprint (none) -> Connector_PinHeader_2.54mm:PinHeader_2x04_P2.54mm_Vertical_SMD
- R3, R5, R6, R7, R8: value R -> 10K
- R4: renamed from R1; value R -> 10K
- gave numbers to parts that had none: 9
- renumbered C13 to C10, C14 to C11, C9 to C12, C10 to C13, C15 to C14, C11 to C15, C12 to C16, C16 to C17, C17 to C19, C1 to C2, C2 to C3, C3 to C4, C6 to C5, C7 to C6, C4 to C7, C5 to C8, C8 to C9, J2 to J1, J1 to J2, R12 to R14, R13 to R15, R11 to R2, R9 to R20, R10 to R21, TP17 to TP30, TP18 to TP31, TP22 to TP32, TP23 to TP33, TP21 to TP34, TP25 to TP36, U3 to U2, U2 to U3
Connections:
- net labels added: LED0, LED1, LED2, LED3, LED4, LED5, LED6, LED7, PB0, PB1, PB2, PB3, PB4, PB5, PB6, PB7
- wire segments 287 -> 330
Other:
- note added: "CARD_DET"
- note added: "CLK/SCLK"
- note added: "CMD/MOSI"
- note added: "D1"
- note added: "D2"
- note added: "D3/CS"
- note added: "DO/MISO"
- note added: "Detection Switch:\n - High when no card present\n - Low when card present"
- note added: "RST_n"
- note added: "SPI Memory Card"
- note added: "Select ROM DOWN"
- note added: "Select ROM UP"
- note removed: "Micro SD Card"
- moved on the sheet: C3, C4, C5, C6, D1, J1, R4, TP1, TP2, TP3, TP4, TP5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

Commit message: Finishing up the peripherals for the FPGA in the schematic, adding the CRESET and CDONE circuits and decoupling for IO power pins.
Parts:
- added C1, C17, C5, C8: 10u, Capacitor_SMD:C_0603_1608Metric, symbol Device:C
- added C10, C19, C2, C6: 1u0, Capacitor_SMD:C_0603_1608Metric, symbol Device:C
- added C13, C20, C3, C7: 100n, Capacitor_SMD:C_0603_1608Metric, symbol Device:C
- added C16, C18, C21: 10n, Capacitor_SMD:C_0603_1608Metric, symbol Device:C
- added D1: LED, LED_SMD:LED_0603_1608Metric, symbol Device:LED
- added FID1, FID2, FID3, FID4: Fiducial, Fiducial:Fiducial_1mm_Mask2mm, symbol Mechanical:Fiducial
- added H1: MountingHole, MountingHole:MountingHole_3.2mm_M3_Pad_Via, symbol Mechanical:MountingHole
- added R12, R18, R5: 10K, Resistor_SMD:R_0603_1608Metric, symbol Device:R
- added R2: R, Resistor_SMD:R_0603_1608Metric, symbol Device:R
- added R3: 1K, Resistor_SMD:R_0603_1608Metric, symbol Device:R
- added TP1, TP18, TP27: TestPoint, TestPoint:TestPoint_Pad_D1.0mm, symbol Connector:TestPoint
- R21: renamed from R16; value 10K -> NP
- R22: renamed from R17; value 10K -> NP
- renumbered C3 to C11, C4 to C12, C5 to C14, C6 to C15, C7 to C22, C8 to C23, C9 to C24, C10 to C25, C11 to C26, C12 to C27, C13 to C28, C14 to C29, C15 to C30, C16 to C31, C17 to C32, C18 to C33, C19 to C34, C1 to C4, C2 to C9, D1 to D2, D2 to D3, D3 to D4, D4 to D5, D5 to D6, D6 to D7, D7 to D8, D8 to D9, R6 to R10, R7 to R11, R8 to R13, R9 to R14, R10 to R15, R11 to R16, R12 to R17, R14 to R19, R15 to R20, R18 to R23, R19 to R24, R20 to R25, R21 to R26, R2 to R4, R3 to R6, R13 to R7, R4 to R8, R5 to R9, SW3 to SW2, SW2 to SW3, TP9 to TP10, TP10 to TP11, TP11 to TP12, TP12 to TP13, TP13 to TP14, TP14 to TP15, TP15 to TP16, TP16 to TP17, TP17 to TP19, TP1 to TP2, TP18 to TP20, TP19 to TP21, TP20 to TP22, TP21 to TP23, TP22 to TP24, TP23 to TP25, TP24 to TP26, TP25 to TP28, TP26 to TP29, TP2 to TP3, TP27 to TP30, TP28 to TP31, TP29 to TP32, TP30 to TP33, TP31 to TP34, TP32 to TP35, TP33 to TP36, TP34 to TP37, TP35 to TP38, TP36 to TP39, TP3 to TP4, TP37 to TP40, TP4 to TP5, TP5 to TP6, TP6 to TP7, TP7 to TP8, TP8 to TP9
Connections:
- wire segments 330 -> 386
Other:
- note added: "1\n<- ~2*Fconf*Ctrace~"
- note added: "Remove JP1 for programming FPGA only\nBridge JP1 for programming FLASH as in normal operation."
- note removed: "RST_n"
- note removed: "Remove JP1 for programming in-circuit emulator only.\nBridge JP1 for programming FLASH as in normal operation."
- moved on the sheet: D6, D7, D8, D9, JP1, R13, R14, R15, R16, R17, R6, R7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

Commit message: Completed a functional version of the schematic and started with basic layout of the components on the PCB.
Parts:
- removed J3: Conn_02x04_Odd_Even, Connector_PinHeader_2.54mm:PinHeader_2x04_P2.54mm_Vertical_SMD, symbol Connector_Generic:Conn_02x04_Odd_Even
- removed TP10, TP11, TP12, TP13, TP14, TP15, TP16, TP17, TP19, TP2, TP20, TP21, TP22, TP23, TP24, TP25, TP26, TP28, TP29, TP3, TP30, TP31, TP32, TP4, TP5, TP6, TP7, TP8, TP9: TestPoint, TestPoint:TestPoint_Pad_D1.0mm, symbol Connector:TestPoint
- added C21: NP, Capacitor_SMD:C_0603_1608Metric, symbol Device:C_Small
- added D2: LED, LED_SMD:LED_0603_1608Metric, symbol Device:LED
- added J3: PMOD, Connector_PinHeader_2.54mm:PinHeader_2x06_P2.54mm_Horizontal, symbol Connector_Generic:Conn_02x06_Top_Bottom
- added J4: Conn_02x05_Odd_Even, Connector_PinHeader_2.54mm:PinHeader_2x05_P2.54mm_Vertical_SMD, symbol Connector_Generic:Conn_02x05_Odd_Even
- added JP1, JP2, JP6: Jumper_NC_Dual, Jumper:SolderJumper-3_P1.3mm_Open_Pad1.0x1.5mm_NumberLabels, symbol Device:Jumper_NC_Dual
- added R11: 1K, Resistor_SMD:R_0603_1608Metric, symbol Device:R
- added R13, R14, R15, R16, R25, R26, R27, R28: 10K, Resistor_SMD:R_0603_1608Metric, symbol Device:R
- added R2: 100R, Resistor_SMD:R_0603_1608Metric, symbol Device:R_Small
- added R3: 10K, Resistor_SMD:R_0603_1608Metric, symbol Device:R_Small
- added R4, R5, R6, R7: 100R, Resistor_SMD:R_0603_1608Metric, symbol Device:R
- added TP1, TP10, TP11, TP12, TP13, TP14, TP15, TP16, TP17, TP18, TP19, TP2, TP20, TP21, TP22, TP23, TP24, TP25, TP26, TP27, TP28, TP29, TP3, TP30, TP31, TP36, TP37, TP38, TP39, TP4, TP41, TP42, TP43, TP44, TP45, TP46, TP47, TP48, TP49, TP5, TP50, TP51, TP52, TP53, TP54, TP55, TP56, TP57, TP58, TP59, TP6, TP60, TP61, TP62, TP63, TP7, TP8, TP9: TestPoint_Probe, TestPoint:TestPoint_Pad_1.0x1.0mm, symbol Connector:TestPoint_Probe
- added TP34, TP35: TestPoint, TestPoint:TestPoint_Pad_1.0x1.0mm, symbol Connector:TestPoint
- CN1: footprint (none) -> iceGDROM:Molex_052602_0579
- TP32: renamed from TP1; footprint TestPoint:TestPoint_Pad_D1.0mm -> TestPoint:TestPoint_Pad_1.0x1.0mm
- TP33: renamed from TP18; footprint TestPoint:TestPoint_Pad_D1.0mm -> TestPoint:TestPoint_Pad_1.0x1.0mm
- TP40: renamed from TP27; footprint TestPoint:TestPoint_Pad_D1.0mm -> TestPoint:TestPoint_Pad_1.0x1.0mm
- renumbered C12 to C10, C8 to C11, C10 to C12, C21 to C22, C22 to C23, C23 to C24, C24 to C25, C25 to C26, C26 to C27, C27 to C28, C28 to C29, C29 to C30, C30 to C31, C31 to C32, C32 to C33, C33 to C34, C34 to C35, C9 to C8, C11 to C9, D9 to D10, D2 to D3, D3 to D4, D4 to D5, D5 to D6, D6 to D7, D7 to D8, D8 to D9, JP1 to JP3, JP2 to JP4, JP3 to JP5, R3 to R10, R6 to R12, R8 to R17, R9 to R18, R10 to R19, R11 to R20, R12 to R21, R5 to R22, R7 to R23, R13 to R24, R14 to R29, R15 to R30, R16 to R31, R17 to R32, R18 to R33, R19 to R34, R20 to R35, R21 to R36, R22 to R37, R23 to R38, R24 to R39, R25 to R40, R26 to R41, R4 to R8, R2 to R9, TP33 to TP64, TP34 to TP65, TP35 to TP66, TP36 to TP67, TP37 to TP68, TP38 to TP69, TP39 to TP70, TP40 to TP71
Connections:
- net labels added: IORDY, PMOD_1, PMOD_2, PMOD_3, PMOD_4, PMOD_5, PMOD_6, PMOD_7, PMOD_8, ROM_DWN, ROM_UP, SDAT, UART_Rx, UART_Tx
- net labels removed: SDA
- wire segments 386 -> 466
- no-connect marks 6 -> 35
Other:
- note removed: "Test Points"
- moved on the sheet: C1, C11, C12, C13, C16, C2, C3, C5, C6, C7, D1, FID1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

Commit message: Split the IDE header into 40+4 due to SMD header availability. Started with layout of the PCB.
Parts:
- removed H1: MountingHole, MountingHole:MountingHole_3.2mm_M3_Pad_Via, symbol Mechanical:MountingHole
- added H1: MountingHole_Pad, MountingHole:MountingHole_3.2mm_M3_Pad_Via, symbol Mechanical:MountingHole_Pad
- added J3: Conn_02x02_Odd_Even, Connector_PinSocket_2.54mm:PinSocket_2x02_P2.54mm_Vertical_SMD, symbol Connector_Generic:Conn_02x02_Odd_Even
- J2: value Conn_02x22_Odd_Even -> Conn_02x20_Odd_Even; footprint Connector_PinHeader_2.54mm:PinHeader_2x22_P2.54mm_Vertical_SMD -> Connector_PinSocket_2.54mm:PinSocket_2x20_P2.54mm_Vertical_SMD; symbol Connector_Generic:Conn_02x22_Odd_Even -> Connector_Generic:Conn_02x20_Odd_Even
- TP1, TP10, TP11, TP12, TP13, TP14, TP15, TP16, TP17, TP18, TP19, TP2, TP20, TP21, TP22, TP23, TP24, TP25, TP26, TP27, TP28, TP29, TP3, TP30, TP31, TP32, TP33, TP34, TP35, TP36, TP37, TP38, TP39, TP4, TP40, TP41, TP42, TP43, TP44, TP45, TP46, TP47, TP48, TP49, TP5, TP50, TP51, TP52, TP53, TP54, TP55, TP56, TP57, TP58, TP59, TP6, TP60, TP61, TP62, TP63, TP7, TP8, TP9: footprint TestPoint:TestPoint_Pad_1.0x1.0mm -> TestPoint:TestPoint_Pad_D1.0mm
- renumbered J3 to J4, J4 to J5

Commit message: Completed functionality of the PCB layout. Still have to do the silkscreen though.
Parts:
- removed C11, C17, C5: 10u, Capacitor_SMD:C_0603_1608Metric, symbol Device:C
- removed C12, C19, C2, C6: 1u0, Capacitor_SMD:C_0603_1608Metric, symbol Device:C
- removed JP2, JP6: Jumper_NC_Dual, Jumper:SolderJumper-3_P1.3mm_Open_Pad1.0x1.5mm_NumberLabels, symbol Device:Jumper_NC_Dual
- removed JP3, JP5: Jumper_NC_Small, Connector_PinHeader_2.54mm:PinHeader_1x02_P2.54mm_Vertical, symbol Device:Jumper_NC_Small
- removed R13, R14, R15, R16, R17, R18, R19, R20, R25, R26, R27, R28, R29, R30, R31, R32, R34, R35, R38, R39: 10K, Resistor_SMD:R_0603_1608Metric, symbol Device:R
- removed R4, R5, R6, R7: 100R, Resistor_SMD:R_0603_1608Metric, symbol Device:R
- removed TP12, TP19: TestPoint_Probe, TestPoint:TestPoint_Pad_D1.0mm, symbol Connector:TestPoint_Probe
- removed TP66, TP67: TestPoint, TestPoint:TestPoint_Pad_D1.0mm, symbol Connector:TestPoint
- added JP2, JP6: Jumper_3_Bridged12, Jumper:SolderJumper-3_P1.3mm_Bridged12_RoundedPad1.0x1.5mm_NumberLabels, symbol Jumper:Jumper_3_Bridged12
- added JP3: SolderJumper_2_Bridged, Jumper:SolderJumper-2_P1.3mm_Open_TrianglePad1.0x1.5mm, symbol Jumper:SolderJumper_2_Bridged
- added JP5: Jumper_NC_Small, Jumper:SolderJumper-2_P1.3mm_Bridged_Pad1.0x1.5mm, symbol Jumper:SolderJumper_2_Bridged
- added RN1, RN3, RN5: 10K, Resistor_SMD:R_Array_Convex_4x0603, symbol iceGDROM:R_Pack04
- added RN2, RN4: R_Pack04, Resistor_SMD:R_Array_Convex_4x0603, symbol Device:R_Pack04
- added RN6: 100R, Resistor_SMD:R_Array_Convex_4x0603, symbol iceGDROM:R_Pack04
- added TP13: TestPoint_Probe, TestPoint:TestPoint_Pad_D1.0mm, symbol Connector:TestPoint_Probe
- added TP19, TP72: TestPoint, symbol Connector:TestPoint
- C1: value 10u -> 100n
- J4: footprint Connector_PinHeader_2.54mm:PinHeader_2x06_P2.54mm_Horizontal -> iceGDROM:PMOD_Host_2x06_P2.54mm_Horizontal
- JP1: footprint Jumper:SolderJumper-3_P1.3mm_Open_Pad1.0x1.5mm_NumberLabels -> Jumper:SolderJumper-3_P1.3mm_Bridged12_RoundedPad1.0x1.5mm
- JP4: footprint Connector_PinHeader_2.54mm:PinHeader_1x02_P2.54mm_Vertical -> Jumper:SolderJumper-2_P1.3mm_Bridged_Pad1.0x1.5mm; symbol Device:Jumper_NC_Small -> Jumper:SolderJumper_2_Bridged
- renumbered TP13 to TP12
Connections:
- net +3V3: now also JP2.1 (A), JP6.1 (A), RN5.5, RN5.6, RN5.7, RN5.8, TP19.1
- net +5V: now also JP2.3 (B), JP6.3 (B)
- net A0: now also U1.D1 (IOL_8B); no longer U1.G3 (IOL_17A)
- net A1: now also U1.E2 (IOL_10A); no longer U1.H3 (IOL_17B)
- net A2: now also U1.D2 (IOL_9A); no longer U1.H1 (IOL_18A)
- net CD_CLK: now also RN6.2
- net CS0n: now also U1.C1 (IOL_5B); no longer U1.J11 (IOR_114)
- net CS1n: now also U1.C2 (IOL_5A); no longer U1.K11 (IOR_115)
- net D0: now also U1.H1 (IOL_18A); no longer U1.B1 (IOL_2A)
- net D1: now also U1.J1 (IOL_23A); no longer U1.B2 (IOL_2B)
- net D10: now also U1.K5 (IOB_79); no longer U1.E2 (IOL_10A)
- net D11: now also U1.K4 (IOB_73); no longer U1.E3 (IOL_10B)
- net D12: now also U1.L2 (IOB_61); no longer U1.F1 (IOL_12A)
- net D13: now also U1.K3 (IOB_63); no longer U1.F2 (IOL_12B)
- net D14: now also U1.K2 (IOL_25A); no longer U1.F4 (IOL_13A)
- net D15: now also U1.H2 (IOL_18B); no longer U1.G2 (IOL_14B)
- net D2: now also U1.K1 (IOL_23B); no longer U1.C4 (IOL_4A)
- net D3: now also U1.L1 (IOB_56); no longer U1.C3 (IOL_4B)
- net D4: now also U1.L3 (IOB_71); no longer U1.C2 (IOL_5A)
- net D5: now also U1.L4 (IOB_72); no longer U1.C1 (IOL_5B)
- net D6: now also U1.L5 (IOB_81_GBIN5); no longer U1.E1 (IOL_8A)
- net D7: now also U1.L7 (IOB_94); no longer U1.D1 (IOL_8B)
- net D8: now also U1.K7 (IOB_89); no longer U1.D2 (IOL_9A)
- net D9: now also U1.K6 (IOB_82_GBIN4); no longer U1.D3 (IOL_9B)
- net DMACKn: now also U1.F2 (IOL_12B); no longer U1.G8 (IOR_118)
- net DMARQ: now also U1.J2 (IOL_25B); no longer U1.H11 (IOR_119)
- net FLASH_CSn: now also JP3.1 (A)
- net FLASH_MISO|IO1: now also JP5.2 (B)
- net FLASH_~RST~|IO3: now also RN5.2
- net FLASH_~WP~|IO2: now also RN5.3
- net FPGA_SCK: now also RN5.1
- net FPGA_SDI: now also JP5.1 (A)
- net GND: now also TP72.1
- net G_RST: now also U1.L8 (IOB_103_CBSEL0); no longer U1.G11 (IOR_129)
- net INTRQ: now also U1.E1 (IOL_8A); no longer U1.G9 (IOR_128)
- net IO_RDY: now also TP29.1, U1.F1 (IOL_12A)
- net LED0: now also U1.A11 (IOT_168), RN2.4 (R4.1); no longer TP11.1, U1.A7 (IOT_192)
- net LED1: now also U1.D10 (IOR_154), RN2.3 (R3.1); no longer TP12.1, U1.A6 (IOT_206)
- net LED2: now also U1.A10 (IOT_170), RN2.2 (R2.1); no longer TP14.1, U1.A5 (IOT_207)
- net LED3: now also U1.B9 (IOT_174), RN2.1 (R1.1); no longer TP15.1, U1.B5 (IOT_208)
- net LED4: now also U1.A9 (IOT_178), RN4.4 (R4.1); no longer TP16.1, U1.A4 (IOT_211)
- net LED5: now also U1.C8 (IOT_179), RN4.3 (R3.1); no longer TP17.1, U1.D5 (IOT_212)
- net LED6: now also U1.B11 (IOR_161), RN4.2 (R2.1); no longer TP18.1, U1.B4 (IOT_219)
- net LED7: now also U1.C11 (IOR_160), RN4.1 (R1.1); no longer U1.B3 (IOT_221)
- net LRCK: now also RN6.3
- net PB0: now also U1.K11 (IOR_115); no longer U1.A11 (IOT_168)
- net PB1: now also U1.B3 (IOT_221); no longer U1.A10 (IOT_170)
- net PB2: now also U1.A3 (IOT_223); no longer U1.C9 (IOT_172)
- net PB3: now also U1.A2 (IOT_222); no longer U1.B9 (IOT_174)
- net PB4: now also U1.B2 (IOL_2B); no longer U1.B8 (IOT_177)
- net PB5: now also U1.A4 (IOT_211); no longer U1.A9 (IOT_178)
- net PB6: now also U1.B4 (IOT_219); no longer U1.C8 (IOT_179)
- net PB7: now also U1.D11 (IOR_152); no longer U1.D7 (IOT_181)
- net PMOD_1: now also U1.A8 (IOT_190), RN1.8; no longer TP36.1, U1.L1 (IOB_56)
- net PMOD_2: now also U1.A7 (IOT_192), RN1.6; no longer TP37.1, U1.J3 (IOB_57)
- net PMOD_3: now also U1.A6 (IOT_206), RN3.8; no longer TP38.1, U1.L2 (IOB_61)
- net PMOD_4: now also U1.A5 (IOT_207), RN3.6; no longer TP39.1, U1.K3 (IOB_63)
- net PMOD_5: now also U1.B8 (IOT_177), RN1.7; no longer TP41.1, U1.J4 (IOB_64)
- net PMOD_6: now also U1.B6 (IOT_198_GBIN0), RN1.5; no longer TP42.1, U1.L3 (IOB_71)
- net PMOD_7: now also U1.B5 (IOT_208), RN3.7; no longer TP43.1, U1.L4 (IOB_72)
- net PMOD_8: now also U1.C4 (IOL_4A), RN3.5; no longer TP44.1, U1.K4 (IOB_73)
- net RDn: now also U1.G2 (IOL_14B); no longer U1.H10 (IOR_116)
- net REFCLK: now also U1.F11 (IOR_140_GBIN3); no longer U1.B6 (IOT_198_GBIN0)
- net ROM_DWN: now also C18.1, R21.1, U1.B1 (IOL_2A); no longer C22.1, R33.1, U1.C7 (IOT_191)
- net ROM_UP: now also C22.1, R33.1, U1.A1 (IOT_225); no longer C18.1, R21.1, U1.A8 (IOT_190)
- net SCK: now also RN6.4
- net SDAT: now also RN6.1
- net UART_Rx: now also U1.J10 (IOR_117); no longer U1.A3 (IOT_223)
- net UART_Tx: now also U1.J11 (IOR_114); no longer U1.A2 (IOT_222)
- net VLOGIC: now also JP2.2 (C)
- net VMOTOR: now also JP6.2 (C)
- net WRn: now also U1.G1 (IOL_14A_GBIN6); no longer U1.J10 (IOR_117)
- net at U1.F10 (IOR_136): now also RN6.8
- net at D3.2 (A): now also TP11.1, RN2.5 (R4.2)
- net at TP64.1, U4.1 (~CS): now also JP3.2 (B), RN5.4
- net at D4.2 (A): now also TP12.1, RN2.6 (R3.2)
- net at D5.2 (A): now also RN2.7 (R2.2), TP13.1
- net at D6.2 (A): now also TP14.1, RN2.8 (R1.2)
- net at D7.2 (A): now also TP15.1, RN4.5 (R4.2)
- net at D8.2 (A): now also TP16.1, RN4.6 (R3.2)
- net at D9.2 (A): now also TP17.1, RN4.7 (R2.2)
- net at D10.2 (A): now also TP18.1, RN4.8 (R1.2)
- net at J4.1 (Pin_1): now also TP36.1, RN1.1
- net at J4.10 (Pin_10): now also TP44.1, RN3.4
- net at J4.2 (Pin_2): now also TP37.1, RN1.3
- net at J4.3 (Pin_3): now also TP38.1, RN3.1
- net at J4.4 (Pin_4): now also TP39.1, RN3.3
- net at J4.7 (Pin_7): now also TP41.1, RN1.2
- net at J4.8 (Pin_8): now also TP42.1, RN1.4
- net at J4.9 (Pin_9): now also TP43.1, RN3.2
- net IORDY: no longer names the net of U1.G10 (IOR_120)
- net IORDY: now also RN6.6; no longer TP29.1
- new net: RN6.7, U1.G11 (IOR_129)
- new net: RN6.5, U1.H11 (IOR_119)
- no-connect marks 35 -> 24
Other:
- moved on the sheet: C21, C24, D1, D3, D4, D5, D6, J4, J5, R2, R3, R36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

Commit message: Finalising the silkscreen & the schematic page
Parts:
- J4: footprint iceGDROM:PMOD_Host_2x06_P2.54mm_Horizontal -> iceGDROM:PMOD_Host_2x06_P2.54mm_Vertical
Connections:
- no-connect marks 24 -> 35
Other:
- note added: "Development "PMOD" Interface"
- note added: "FPGA"
- note added: "IDE Header Settings"
- note added: "PCB"
- moved on the sheet: C1, C13, C16, C18, C20, C21, C22, C24, C3, C7, D1, D2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
