File: pcb/USB PMOD/USB PMOD.kicad_pcb (KiCad board)
At the start: 2 copper layers, 15 x 44.5 mm, 6 parts, among them J1 USB_B_Mini, J2 PMOD

Commit message: Deleting backup files from git repository, and updating the USB PMOD board to latest nightly build.
Other:
- net class Default removed
